File: fcmpill.kicad_pcb (KiCad board)
At the start: 2 copper layers, 19.7 x 43.2 mm, 43 parts, among them J1 Conn_01x15_Socket, J2 Conn_01x15_Socket, J3 Conn_01x04_Pin, J4 USB_B_Micro, J5 Conn_01x03_Pin, SW1 SW_DIP_x02, SW2 KXT331LHS, U1 STM32F103C8Tx, U2 AP63205WU, U3 AP63203WU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

Commit message: 20250915
Parts:
- C1, C10, C14, C15, C16, C17, C18, C2, C3, C4, C5, C6, C7, C8, C9: footprint Capacitor_SMD:C_0201_0603Metric -> Capacitor_SMD:C_0402_1005Metric
- D3: value XL-0201SURC -> XL-1005SURC; footprint LED_SMD:LED_0201_0603Metric -> LED_SMD:LED_0402_1005Metric
- R4: footprint Resistor_SMD:R_0201_0603Metric -> Resistor_SMD:R_0402_1005Metric
- Y1: value X32258MOB4SI -> SX2M8.000M20F30TNN; footprint Crystal:Crystal_SMD_3225-4Pin_3.2x2.5mm -> Crystal:Crystal_SMD_2520-4Pin_2.5x2.0mm
- moved D3 1.50 mm to (135.1, 72.4)
- moved C18 0.68 mm to (145.7, 66.9)
- moved C14 0.57 mm to (134.3, 67.1)
- moved C17 0.55 mm to (144.8, 66.9)
- moved L2 0.51 mm to (136.3, 67.2)
- moved C3 0.49 mm to (137.2, 71.4), turned to 180 degrees
- moved C4 0.47 mm to (135.1, 71.4)
- moved Y1 0.44 mm to (136.5, 69.4)
- moved D2 0.43 mm to (143.9, 67.0)
- moved C15 0.39 mm to (143.0, 67.3)
- moved R4 0.34 mm to (135.1, 73.4)
- moved L1 0.31 mm to (141.0, 67.1)
- moved Y2 0.27 mm to (140.6, 69.5)
- moved C13 0.27 mm to (139.0, 65.7)
- moved C11 0.22 mm to (144.5, 64.4)
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Routing:
- net GND: track 70.8 -> 81.9 mm, vias 73 -> 80
- net VDD: track 57.9 -> 63.0 mm
- net 5V: track 47.4 -> 49.4 mm
- net RESET: track 35.8 -> 37.4 mm
- net PB0: track 5.53 -> 6.26 mm
- net PA3: track 10.0 -> 9.50 mm
- net RTCIN: track 8.00 -> 7.78 mm, vias 2 -> 0
Other:
- board text added: "5V Vin 3V3"
